File: pcb/k60.brd (EAGLE design)
At the start: 15.6 x 16.4 mm, 129 parts, among them U1 USBLC6-2P6, U2 ATMEGA32U4-AU, X1 S4B-ZR

Commit message: aligned missaligned keys
Parts:
- moved U2 200.9 mm to (14.2, -95.0)
- moved 6,5 134.7 mm to (216.1, -76.0)
- moved 1,1 134.4 mm to (0.00, 0.00)
- moved 1,2 134.4 mm to (4.75, -19.0)
- moved 10,1 134.4 mm to (171.0, 0.00)
- moved 10,2 134.4 mm to (180.5, -19.0)
- moved 10,3 134.4 mm to (185.2, -38.0)
- moved 10,4 134.4 mm to (194.8, -57.0)
- moved 11,1 134.4 mm to (190.0, 0.00)
- moved 11,2 134.4 mm to (199.5, -19.0)
- moved 11,3 134.4 mm to (204.2, -38.0)
- moved 11,4 134.4 mm to (213.8, -57.0)
- moved 12,1 134.4 mm to (209.0, 0.00)
- moved 12,2 134.4 mm to (218.5, -19.0)
- moved 12,3 134.4 mm to (223.2, -38.0)
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
Commit message: fixed board dimensions, mx_switch
original mx_switch component was using layer 20 (Dimension)
layer 20 is used to determine pcb surface
moved outline from layer 20 to layer 51 (tDocu)

hint:
to update component lib add new component from this lib in .sch file

added rough pcb dimension and mounting points for stabilizers
TODO: add mounting case mounting points
Parts:
- removed QF1: 16M20AUM1, crystal:UM1
- moved U2 60.1 mm to (71.2, -76.0), turned to 180 degrees
- moved X1 55.6 mm to (102.0, -72.3)
- moved R1 46.8 mm to (85.3, -72.7)
- moved R2 46.8 mm to (85.3, -77.8)
- moved U1 25.6 mm to (84.9, -83.1)
- moved D53 25.5 mm to (241.3, -55.7)
- moved D41 23.5 mm to (245.6, -37.1)
- moved C1 17.1 mm to (80.5, -83.1)
- moved D28 14.0 mm to (252.6, -18.3)
- moved D62 12.0 mm to (255.3, -75.1)
- moved D29 7.00 mm to (17.2, -36.6)
- moved D14 5.52 mm to (248.2, 0.50)
- moved D27 5.50 mm to (246.1, -18.3)
- moved D50 5.00 mm to (184.3, -54.7)
- moved D52 5.00 mm to (222.1, -54.7)
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Connections:
- removed net N$2: U2.17
- removed net N$3: U2.16
Routing:
- net N$81: track 2964.0 -> 0.00 mm
Other:
- board size 15.6 x 16.4 mm -> 285 x 95 mm

Commit message: changed lib to custom k60 lib
Parts:
- removed U2: ATMEGA32U4-AU, SnapEDA-Library:QFP80P1200X1200X120-44N
- removed X1: S4B-ZR, con-jst:S4B-ZR
- added C2: CL21C220JBANNNC, k60:CAPC2012X140N
- added C3: CL21B105KBFNNNE, k60:CL21B105KBFNNNE_CAPC2012X140N
- added D54: BAV21W-7-F, k60:SOD3715X135N
- added J1: SM04B-SRSS-TB(LF)(SN), k60:JST_SM04B-SRSS-TB(LF)(SN)
- added R3, R4: 1623158-1, k60:RESC2012X65N
- added Y1: X322516MLB4SI, k60:OSC_X322516MLB4SI
- C1: value GRM155R6YA105KE11D -> CL21C220JBANNNC; device SnapEDA-Library:CAPC1005X60N -> k60:CAPC2012X140N
- D1, D10, D11, D12, D13, D14, D15, D16, D17, D18, D19, D2, D20, D21, D22, D23, D24, D25, D26, D27, D28, D29, D3, D30, D31, D32, D33, D34, D35, D36, D37, D38, D39, D4, D40, D41, D42, D43, D44, D45, D46, D47, D48, D49, D5, D50, D51, D52, D53, D55, D56, D57, D58, D59, D6, D60, D61, D7, D8, D9: value 1N4148WS -> BAV21W-7-F; device SnapEDA-Library:SODFL2512X100N -> k60:SOD3715X135N
- D62: value 1N4148WS -> USBLC6-2SC6; device SnapEDA-Library:SODFL2512X100N -> k60:SOT95P280X145-6N
- R1, R2: value 350222RFT -> 0805W8F1002T5E; device SnapEDA-Library:RESC5025X120N -> k60:RESC2012X60N
- U1: value USBLC6-2P6 -> ATMEGA32U4-AU; device SnapEDA-Library:SOT50P160X60-6N -> k60:QFP80P1200X1200X120-44N
- moved D62 640.0 mm to (-14.2, -655.5), flipped to the top, turned to 0 degrees
- moved D61 637.2 mm to (-4.75, -660.2), flipped to the top, turned to 0 degrees
- moved R1 634.8 mm to (-47.5, -693.5), flipped to the top
- moved R2 634.5 mm to (-47.5, -698.2), flipped to the top
- moved D60 619.8 mm to (-4.75, -650.8), flipped to the top, turned to 0 degrees
- moved U1 610.7 mm to (-47.5, -679.2), flipped to the top
- moved D59 601.9 mm to (-4.75, -641.2), flipped to the top, turned to 0 degrees
- moved C1 597.6 mm to (-33.2, -669.8), flipped to the top
- moved D53 583.0 mm to (-4.75, -584.2), flipped to the top, turned to 0 degrees
- moved D58 572.8 mm to (-4.75, -631.8), flipped to the top, turned to 0 degrees
- moved D52 567.3 mm to (-4.75, -574.8), flipped to the top, turned to 0 degrees
- moved D51 551.4 mm to (-4.75, -565.2), flipped to the top, turned to 0 degrees
- moved D57 549.8 mm to (-4.75, -622.2), flipped to the top, turned to 0 degrees
- moved D56 537.7 mm to (-4.75, -612.8), flipped to the top, turned to 0 degrees
- moved D50 535.5 mm to (-4.75, -555.8), flipped to the top, turned to 0 degrees
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Connections:
- removed net D+: R2.2, U2.4
- removed net D-: R1.2, U2.3
- removed net N$1: R2.1, U1.6
- removed net N$4: R1.1, U1.4
- removed net N$5: U1.1, X1.3
- removed net N$6: U1.3, X1.2
- removed net N$7: C1.1, U2.6
- new net AVCC: U1.44
- new net AVCC_2: U1.24
- new net UCAP: U1.6
- new net UVCC: U1.2
- new net VBUS: D62.5
- new net VCC_2: U1.14
- net COL1: no longer U2.8
- net COL10: no longer U2.19
- net COL11: no longer U2.20
- net COL12: no longer U2.21
- net COL13: no longer U2.25
- net COL14: no longer U2.22
- net COL2: no longer U2.9
- net COL3: no longer U2.10
- net COL4: no longer U2.11
- net COL5: no longer U2.28
- net COL6: no longer U2.29
- net COL7: no longer U2.30
- net COL8: no longer U2.12
- net COL9: no longer U2.18
- net GND: now also D62.2, Y1.2, Y1.4; no longer C1.2, U1.2, U2.15, U2.23, U2.35, U2.43, U2.5, X1.4
- net N$69: now also D61.A; no longer D55.A
- net N$70: now also D60.A; no longer D56.A
- net N$71: now also D59.A; no longer D57.A
- net N$73: now also D57.A; no longer D59.A
- net N$74: now also D56.A; no longer D60.A
- net N$75: now also D55.A; no longer D61.A
- net N$76: now also D54.A; no longer D62.A
- net ROW1: no longer U2.41
- net ROW2: no longer U2.40
- net ROW3: no longer U2.39
- net ROW4: no longer U2.38
- net ROW5: now also D54.C; no longer D62.C, U2.37
- net VCC: now also U1.34; no longer U1.5, U2.14, U2.2, U2.24, U2.34, U2.44, X1.1

Commit message: moved to positive coordinates
Parts:
- moved 1,1 96.9 mm to (19.0, 95.0)
- moved 1,2 96.9 mm to (23.8, 76.0)
- moved 1,3 96.9 mm to (26.1, 57.0)
- moved 1,4 96.9 mm to (30.9, 38.0)
- moved 1,5 96.9 mm to (21.4, 19.0)
- moved 10,1 96.9 mm to (190.0, 95.0)
- moved 10,2 96.9 mm to (199.5, 76.0)
- moved 10,3 96.9 mm to (204.2, 57.0)
- moved 10,4 96.9 mm to (213.8, 38.0)
- moved 11,1 96.9 mm to (209.0, 95.0)
- moved 11,2 96.9 mm to (218.5, 76.0)
- moved 11,3 96.9 mm to (223.2, 57.0)
- moved 11,4 96.9 mm to (232.8, 38.0)
- moved 12,1 96.9 mm to (228.0, 95.0)
- moved 12,2 96.9 mm to (237.5, 76.0)
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
Commit message: schematic cleanup, connected important compoonents
added power stabilization (10uF, 1uF)
Parts:
- added C4: CL21A106KAYNNNE, k60:CAPC2012X135N
- added C5, C6, C7: CC0805KRX7R9BB104, k60:CAPC2012X70
- added R5: NSMD050-24V, k60:RESC3115X65N
- added S1: TS-1187A-B-A-B, k60:SW_TS-1187A-B-A-B
- moved R2 741.8 mm to (120.5, 24.2), flipped to the bottom, turned to 270 degrees
- moved R4 741.2 mm to (97.0, 30.5), flipped to the bottom, turned to 180 degrees
- moved R3 737.8 mm to (97.0, 28.0), flipped to the bottom, turned to 180 degrees
- moved C3 730.7 mm to (103.8, 29.0), flipped to the bottom
- moved R1 721.2 mm to (104.5, 11.5), flipped to the bottom, turned to 180 degrees
- moved C2 718.5 mm to (116.5, 23.5), flipped to the bottom
- moved U1 715.5 mm to (104.0, 20.0), flipped to the bottom, turned to 270 degrees
- moved C1 703.4 mm to (116.5, 17.5), flipped to the bottom
- moved J1 693.9 mm to (84.8, 28.2), flipped to the bottom, turned to 90 degrees
- moved D62 692.5 mm to (91.0, 29.0), flipped to the bottom
- moved Y1 690.4 mm to (116.5, 20.5), flipped to the bottom, turned to 90 degrees
- moved D61 680.1 mm to (30.0, 19.0), flipped to the bottom, turned to 90 degrees
- moved D57 679.5 mm to (220.0, 19.0), flipped to the bottom, turned to 90 degrees
- moved D55 679.0 mm to (267.0, 19.0), flipped to the bottom, turned to 90 degrees
- moved D56 679.0 mm to (244.0, 19.0), flipped to the bottom, turned to 90 degrees
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Connections:
- removed net AVCC: U1.44
- removed net AVCC_2: U1.24
- removed net UCAP: U1.6
- removed net UVCC: U1.2
- removed net VCC: U1.34
- removed net VCC_2: U1.14
- new net +5V: C4.2, C5.2, C6.2, C7.2, R2.2, R5.2, U1.14, U1.2, U1.24, U1.34, U1.44, U1.7
- new net D+: D62.1, D62.6, J1.3, R4.1
- new net D-: D62.3, D62.4, J1.2, R3.1
- new net MCU_D+: R4.2, U1.4
- new net MCU_D-: R3.2, U1.3
- new net N$3: C3.1, U1.6
- new net N$4: R1.1, U1.33
- new net RESET: R2.1, S1.A, S1.B, U1.13
- new net XTAL1: C1.2, U1.17, Y1.1
- new net XTAL2: C2.2, U1.16, Y1.3
- net COL1: now also U1.41
- net COL10: now also U1.27
- net COL11: now also U1.29
- net COL12: now also U1.30
- net COL13: now also U1.12
- net COL14: now also U1.39
- net COL2: now also U1.40
- net COL3: now also U1.18
- net COL4: now also U1.19
- net COL5: now also U1.20
- net COL6: now also U1.21
- net COL7: now also U1.25
- net COL8: now also U1.22
- net COL9: now also U1.26
- net GND: now also C1.1, C2.1, C3.2, C4.1, C5.1, C6.1, C7.1, J1.4, R1.2, S1.C, S1.D, U1.15, U1.23, U1.35, U1.43, U1.5
- net ROW1: now also U1.8
- net ROW2: now also U1.9
- net ROW3: now also U1.10
- net ROW4: now also U1.11
- net ROW5: now also U1.28
- net VBUS: now also J1.1, R5.1
Routing:
- net +5V: track 0.00 -> 31.7 mm
- net RESET: track 0.00 -> 25.0 mm
- net GND: track 0.00 -> 24.2 mm
- net VBUS: track 0.00 -> 10.3 mm
- net XTAL1: track 0.00 -> 9.87 mm
- net D+: track 0.00 -> 9.69 mm
- net XTAL2: track 0.00 -> 9.22 mm
- net D-: track 0.00 -> 9.11 mm
- net MCU_D+: track 0.00 -> 7.23 mm
- net MCU_D-: track 0.00 -> 5.29 mm
- net N$3: track 0.00 -> 3.53 mm
