File: pcb/k60.sch (EAGLE design)
At the start: 129 parts, among them U1 USBLC6-2P6, U2 ATMEGA32U4-AU, X1 S4B-ZR

Commit message: fixed board dimensions, mx_switch
original mx_switch component was using layer 20 (Dimension)
layer 20 is used to determine pcb surface
moved outline from layer 20 to layer 51 (tDocu)

hint:
to update component lib add new component from this lib in .sch file

added rough pcb dimension and mounting points for stabilizers
TODO: add mounting case mounting points
Parts:
- removed QF1: 16M20AUM1, crystal:16M20AUM1
Connections:
- removed net N$2: U2.XTAL1
- removed net N$3: U2.XTAL2
Changed lines of the file:
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@@
 <part name="R2" library="SnapEDA-Library" deviceset="350222RFT" device=""/>
 <part name="C1" library="SnapEDA-Library" deviceset="GRM155R6YA105KE11D" device=""/>
-<part name="QF1" library="crystal" library_urn="urn:adsk.eagle:library:204" deviceset="16M20AUM1" device="" package3d_urn="urn:adsk.eagle:package:12117/1"/>
 </parts>
 <sheets>
@@
 <attribute name="NAME" x="-83.82" y="-19.04906875" size="1.77843125" layer="95"/>
 <attribute name="VALUE" x="-83.82" y="-27.94848125" size="1.78096875" layer="96"/>
-</instance>
-<instance part="QF1" gate="G$1" x="-101.6" y="132.08" smashed="yes">
-<attribute name="NAME" x="-99.06" y="133.096" size="1.778" layer="95"/>
-<attribute name="VALUE" x="-99.06" y="129.54" size="1.778" layer="96"/>
 </instance>
 </instances>
@@
 </segment>
 </net>
-<net name="N$2" class="0">
-<segment>
-<pinref part="U2" gate="G$1" pin="XTAL1"/>
-<wire x1="-119.38" y1="22.86" x2="-124.46" y2="22.86" width="0.1524" layer="91"/>
-<wire x1="-124.46" y1="22.86" x2="-124.46" y2="132.08" width="0.1524" layer="91"/>
-</segment>
-</net>
-<net name="N$3" class="0">
-<segment>
-<pinref part="U2" gate="G$1" pin="XTAL2"/>
-<wire x1="-88.9" y1="22.86" x2="-68.58" y2="22.86" width="0.1524" layer="91"/>
-<wire x1="-68.58" y1="22.86" x2="-68.58" y2="104.14" width="0.1524" layer="91"/>
-</segment>
-</net>

Commit message: changed lib to custom k60 lib
Parts:
- removed U2: ATMEGA32U4-AU, SnapEDA-Library:ATMEGA32U4-AU
- removed X1: S4B-ZR, con-jst:S4B-ZR
- added C2: CL21C220JBANNNC, k60:CL21C220JBANNNC
- added C3: CL21B105KBFNNNE, k60:CL21B105KBFNNNE
- added D54: BAV21W-7-F, k60:BAV21W-7-F
- added J1: SM04B-SRSS-TB(LF)(SN), k60:SM04B-SRSS-TB(LF)(SN)
- added R3, R4: 1623158-1, k60:1623158-1
- added Y1: X322516MLB4SI, k60:X322516MLB4SI
- C1: value GRM155R6YA105KE11D -> CL21C220JBANNNC; device SnapEDA-Library:GRM155R6YA105KE11D -> k60:CL21C220JBANNNC
- D1, D10, D11, D12, D13, D14, D15, D16, D17, D18, D19, D2, D20, D21, D22, D23, D24, D25, D26, D27, D28, D29, D3, D30, D31, D32, D33, D34, D35, D36, D37, D38, D39, D4, D40, D41, D42, D43, D44, D45, D46, D47, D48, D49, D5, D50, D51, D52, D53, D55, D56, D57, D58, D59, D6, D60, D61, D7, D8, D9: value 1N4148WS -> BAV21W-7-F; device SnapEDA-Library:1N4148WS -> k60:BAV21W-7-F
- D62: value 1N4148WS -> USBLC6-2SC6; device SnapEDA-Library:1N4148WS -> k60:USBLC6-2SC6
- R1, R2: value 350222RFT -> 0805W8F1002T5E; device SnapEDA-Library:350222RFT -> k60:0805W8F1002T5E
- U1: value USBLC6-2P6 -> ATMEGA32U4-AU; device SnapEDA-Library:USBLC6-2P6 -> k60:ATMEGA32U4-AU
Connections:
- removed net D+: R2.2, U2.D+
- removed net D-: R1.2, U2.D-
- removed net GND: C1.2, U1.GND, U2.GND, U2.UGND, X1-4.1
- removed net N$1: R2.1, U1.I/O1_2
- removed net N$4: R1.1, U1.I/O2_2
- removed net N$5: U1.I/O1_1, X1-3.1
- removed net N$6: U1.I/O2_1, X1-2.1
- removed net N$7: C1.1, U2.UCAP
- removed net VCC: U1.VBUS, U2.AVCC, U2.UVCC, U2.VCC, X1-1.1
- new net N$68: D54.A
- net COL1: no longer U2.PB0
- net COL10: no longer U2.PD1
- net COL11: no longer U2.PD2
- net COL12: no longer U2.PD3
- net COL13: no longer U2.PD4
- net COL14: no longer U2.PD5
- net COL2: no longer U2.PB1
- net COL3: no longer U2.PB2
- net COL4: no longer U2.PB3
- net COL5: no longer U2.PB4
- net COL6: no longer U2.PB5
- net COL7: no longer U2.PB6
- net COL8: no longer U2.PB7
- net COL9: no longer U2.PD0
- net N$69: now also D61.A
- net N$70: now also D60.A
- net N$71: now also D59.A
- net N$73: now also D57.A
- net N$74: now also D56.A
- net N$75: now also D55.A
- net N$76: now also D54.A
- net ROW1: no longer U2.PF0
- net ROW2: no longer U2.PF1
- net ROW3: no longer U2.PF4
- net ROW4: now also D54.C; no longer U2.PF5
- net ROW5: now also D54.C; no longer U2.PF6
Other:
- moved on the sheet: C1, D55, D56, D57, D59, D60, D61, R1, R2

Commit message: schematic cleanup, connected important compoonents
added power stabilization (10uF, 1uF)
Parts:
- added C4: CL21A106KAYNNNE, k60:CL21A106KAYNNNE
- added C5, C6, C7: CC0805KRX7R9BB104, k60:CC0805KRX7R9BB104
- added R5: NSMD050-24V, k60:NSMD050-24V
- added S1: TS-1187A-B-A-B, k60:TS-1187A-B-A-B
Connections:
- new net +5V: C4.2, C5.2, C6.2, C7.2, R2.2, R5.2, U1.AVCC, U1.AVCC_2, U1.UVCC, U1.VBUS, U1.VCC, U1.VCC_2
- new net D+: D62.I/O1, J1.3, R4.1
- new net D-: D62.I/O2, J1.2, R3.1
- new net GND: C1.1, C2.1, C3.2, C4.1, C5.1, C6.1, C7.1, D62.GND, J1.4, R1.2, S1.NO, U1.GND, U1.GND_2, U1.GND_3, U1.GND_4, U1.UGND, Y1.GND
- new net MCU_D+: R4.2, U1.D+
- new net MCU_D-: R3.2, U1.D-
- new net N$3: C3.1, U1.UCAP
- new net N$4: R1.1, U1.PE2
- new net RESET: R2.1, S1.COM, U1.~RESET
- new net VBUS: D62.VBUS, J1.1, R5.1
- new net XTAL1: C1.2, U1.XTAL1, Y1.1
- new net XTAL2: C2.2, U1.XTAL2, Y1.3
- net COL1: now also S1.1, U1.PF0
- net COL10: now also U1.PD7
- net COL11: now also U1.PB5
- net COL12: now also U1.PB6
- net COL13: now also U1.PB7
- net COL14: now also U1.PF4
- net COL2: now also U1.PF1
- net COL3: now also U1.PD0
- net COL4: now also U1.PD1
- net COL5: now also U1.PD2
- net COL6: now also U1.PD3
- net COL7: now also U1.PD4
- net COL8: now also U1.PD5
- net COL9: now also U1.PD6
- net N$15: now also S1.2
- net ROW1: now also U1.PB0
- net ROW2: now also U1.PB1
- net ROW3: now also U1.PB2
- net ROW4: now also U1.PB3
- net ROW5: now also U1.PB4
Other:
- note added: "Clock"
- note added: "ESD protection"
- note added: "Fuse"
- note added: "Key matrix"
- note added: "Microcontroller"
- note added: "Reset button"
- note added: "USB Connection"
- moved on the sheet: 1,1, 1,2, 1,3, 1,4, 1,5, 10,1, 10,2, 10,3, 10,4, 11,1, 11,2, 11,3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
